Commit message: change effort from 23.7 to 18.0

File: urdf/RCV8.urdf (robot description, URDF)
Before this commit: robot RCV8, 17 links, 16 joints
Joints:
- joint FL_calf_joint: limit lower=-2.72 upper=-0.84 effort=23.7 velocity=30 -> lower=-2.72 upper=-0.84 effort=18.0 velocity=30
- joint FL_hip_joint: limit lower=-1.05 upper=1.05 effort=23.7 velocity=30 -> lower=-1.05 upper=1.05 effort=18.0 velocity=30
- joint FL_thigh_joint: limit lower=-1.57 upper=3.49 effort=23.7 velocity=30 -> lower=-1.57 upper=3.49 effort=18.0 velocity=30
- joint FR_calf_joint: limit lower=-2.72 upper=-0.84 effort=23.7 velocity=30 -> lower=-2.72 upper=-0.84 effort=18.0 velocity=30
- joint FR_hip_joint: limit lower=-1.05 upper=1.05 effort=23.7 velocity=30 -> lower=-1.05 upper=1.05 effort=18.0 velocity=30
- joint FR_thigh_joint: limit lower=-1.57 upper=3.49 effort=23.7 velocity=30 -> lower=-1.57 upper=3.49 effort=18.0 velocity=30
- joint RL_calf_joint: limit lower=-2.72 upper=-0.84 effort=23.7 velocity=30 -> lower=-2.72 upper=-0.84 effort=18.0 velocity=30
- joint RL_hip_joint: limit lower=-1.05 upper=1.05 effort=23.7 velocity=30 -> lower=-1.05 upper=1.05 effort=18.0 velocity=30
- joint RL_thigh_joint: limit lower=-0.52 upper=4.54 effort=23.7 velocity=30 -> lower=-0.52 upper=4.54 effort=18.0 velocity=30
- joint RR_calf_joint: limit lower=-2.72 upper=-0.84 effort=23.7 velocity=30 -> lower=-2.72 upper=-0.84 effort=18.0 velocity=30
- joint RR_hip_joint: limit lower=-1.05 upper=1.05 effort=23.7 velocity=30 -> lower=-1.05 upper=1.05 effort=18.0 velocity=30
- joint RR_thigh_joint: limit lower=-0.52 upper=4.54 effort=23.7 velocity=30 -> lower=-0.52 upper=4.54 effort=18.0 velocity=30
